Commit message: 完成casadi在线优化的代码嵌入，但是存在问题，效果看起来很差

File: phc/data/assets/robot/noetix_n2/urdf/N2.urdf (robot description, URDF)
Before this commit: robot N2, 21 links, 20 joints
Links:
- removed link R_arm_hand_link
- added link R_arm_hand_Link, mass 0.17711; collision mesh filename=/home/djh/PHC/phc/data/assets/robot/noetix_n2/meshes/r_arm_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; visual mesh filename=/home/djh/PHC/phc/data/assets/robot/noetix_n2/meshes/r_arm_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
Joints:
- joint L_arm_hand_joint: limit lower=0 upper=0 effort=36 velocity=1000 -> lower=0.0 upper=0.0 effort=36 velocity=1000
- joint R_arm_hand_joint: child R_arm_hand_link -> R_arm_hand_Link; limit (none) -> lower=0.0 upper=0.0 effort=36 velocity=1000
